File: klasesdarbs/ONE_TRAN_AMP.kicad_pcb (KiCad board)
At the start: 2 copper layers, 52.1 x 30.5 mm, 11 parts, among them J1 Signal in, J2 Signal out, J3 Power, Q1 BC547

Commit message: gerbers
Parts:
- added G***: LOGO, Battery_holders:BrEE_LOGO_0_5_inch, F.Cu at (130.8, 105.4)
